File: Firmware 102/Hardware/DC801 Shield/DC801 Shield.sch (KiCad schematic (older format))
At the start: 13 parts, among them SW1 SW_Push, SW2 SW_Push

Commit message: Finished routing, adding images
Parts:
- removed R2, R3, R4, R5: 150, Resistors_SMD:R_0805, symbol device:R
- added R? (x10): 150, Resistors_SMD:R_0805, symbol device:R
Connections:
- wire segments 51 -> 66
