File: Firmware 102/Hardware/DC801 Shield/DC801 Shield.kicad_pcb (KiCad board)
At the start: 2 copper layers, 53.4 x 68.6 mm, 11 parts

Commit message: Finished routing, adding images
Parts:
- added R1: 150, Resistors_SMD:R_0805, F.Cu at (120.0, 78.0)
- added R10: 150, Resistors_SMD:R_0805, F.Cu at (148.3, 87.2)
- added R6: 150, Resistors_SMD:R_0805, F.Cu at (155.0, 74.0)
- added R7: 150, Resistors_SMD:R_0805, F.Cu at (145.5, 94.5)
- added R8: 150, Resistors_SMD:R_0805, F.Cu at (129.2, 94.5)
- added R9: 150, Resistors_SMD:R_0805, F.Cu at (127.1, 86.8)
- added REF**: SolderWirePad_single_1mmDrill, Wire_Pads:SolderWirePad_single_1mmDrill, F.Cu at (152.0, 120.4)
- added REF**: SolderWirePad_single_1mmDrill, Wire_Pads:SolderWirePad_single_1mmDrill, F.Cu at (129.2, 120.4)
- added REF**: SolderWirePad_single_1mmDrill, Wire_Pads:SolderWirePad_single_1mmDrill, F.Cu at (160.0, 90.9)
- added REF**: SolderWirePad_single_1mmDrill, Wire_Pads:SolderWirePad_single_1mmDrill, F.Cu at (160.0, 88.4)
- added REF**: SolderWirePad_single_1mmDrill, Wire_Pads:SolderWirePad_single_1mmDrill, F.Cu at (160.0, 85.8)
- added REF**: SolderWirePad_single_1mmDrill, Wire_Pads:SolderWirePad_single_1mmDrill, F.Cu at (117.1, 130.6)
- added REF**: SolderWirePad_single_1mmDrill, Wire_Pads:SolderWirePad_single_1mmDrill, F.Cu at (117.1, 128.1)
- added REF**: SolderWirePad_single_1mmDrill, Wire_Pads:SolderWirePad_single_1mmDrill, F.Cu at (117.1, 125.5)
- added REF**: SolderWirePad_single_1mmDrill, Wire_Pads:SolderWirePad_single_1mmDrill, F.Cu at (117.1, 123.0)
- added REF**: SolderWirePad_single_1mmDrill, Wire_Pads:SolderWirePad_single_1mmDrill, F.Cu at (117.1, 120.5)
- added REF**: SolderWirePad_single_1mmDrill, Wire_Pads:SolderWirePad_single_1mmDrill, F.Cu at (117.1, 117.9)
- added REF**: SolderWirePad_single_1mmDrill, Wire_Pads:SolderWirePad_single_1mmDrill, F.Cu at (117.1, 112.9)
- added REF**: SolderWirePad_single_1mmDrill, Wire_Pads:SolderWirePad_single_1mmDrill, F.Cu at (126.6, 120.4)
- added REF**: SolderWirePad_single_1mmDrill, Wire_Pads:SolderWirePad_single_1mmDrill, F.Cu at (117.1, 110.3)
- added REF**: SolderWirePad_single_1mmDrill, Wire_Pads:SolderWirePad_single_1mmDrill, F.Cu at (117.1, 107.8)
- added REF**: SolderWirePad_single_1mmDrill, Wire_Pads:SolderWirePad_single_1mmDrill, F.Cu at (117.1, 105.3)
- added REF**: SolderWirePad_single_1mmDrill, Wire_Pads:SolderWirePad_single_1mmDrill, F.Cu at (117.1, 102.7)
- added REF**: SolderWirePad_single_1mmDrill, Wire_Pads:SolderWirePad_single_1mmDrill, F.Cu at (117.1, 100.2)
- added REF**: SolderWirePad_single_1mmDrill, Wire_Pads:SolderWirePad_single_1mmDrill, F.Cu at (117.1, 97.6)
- added REF**: SolderWirePad_single_1mmDrill, Wire_Pads:SolderWirePad_single_1mmDrill, F.Cu at (117.1, 95.1)
- added REF**: SolderWirePad_single_1mmDrill, Wire_Pads:SolderWirePad_single_1mmDrill, F.Cu at (152.0, 105.2)
- added REF**: SolderWirePad_single_1mmDrill, Wire_Pads:SolderWirePad_single_1mmDrill, F.Cu at (149.5, 105.2)
- added REF**: SolderWirePad_single_1mmDrill, Wire_Pads:SolderWirePad_single_1mmDrill, F.Cu at (147.0, 105.2)
- added REF**: SolderWirePad_single_1mmDrill, Wire_Pads:SolderWirePad_single_1mmDrill, F.Cu at (144.4, 105.2)
- added REF**: SolderWirePad_single_1mmDrill, Wire_Pads:SolderWirePad_single_1mmDrill, F.Cu at (141.9, 105.2)
- added REF**: SolderWirePad_single_1mmDrill, Wire_Pads:SolderWirePad_single_1mmDrill, F.Cu at (139.3, 105.2)
- added REF**: SolderWirePad_single_1mmDrill, Wire_Pads:SolderWirePad_single_1mmDrill, F.Cu at (136.8, 105.2)
- added REF**: SolderWirePad_single_1mmDrill, Wire_Pads:SolderWirePad_single_1mmDrill, F.Cu at (134.3, 105.2)
- added REF**: SolderWirePad_single_1mmDrill, Wire_Pads:SolderWirePad_single_1mmDrill, F.Cu at (149.5, 120.4)
- added REF**: SolderWirePad_single_1mmDrill, Wire_Pads:SolderWirePad_single_1mmDrill, F.Cu at (131.7, 105.2)
- added REF**: SolderWirePad_single_1mmDrill, Wire_Pads:SolderWirePad_single_1mmDrill, F.Cu at (129.2, 105.2)
- added REF**: SolderWirePad_single_1mmDrill, Wire_Pads:SolderWirePad_single_1mmDrill, F.Cu at (126.6, 105.2)
- added REF**: SolderWirePad_single_1mmDrill, Wire_Pads:SolderWirePad_single_1mmDrill, F.Cu at (124.1, 120.4)
- added REF**: SolderWirePad_single_1mmDrill, Wire_Pads:SolderWirePad_single_1mmDrill, F.Cu at (152.0, 117.9)
- added REF**: SolderWirePad_single_1mmDrill, Wire_Pads:SolderWirePad_single_1mmDrill, F.Cu at (149.5, 117.9)
- added REF**: SolderWirePad_single_1mmDrill, Wire_Pads:SolderWirePad_single_1mmDrill, F.Cu at (147.0, 117.9)
- added REF**: SolderWirePad_single_1mmDrill, Wire_Pads:SolderWirePad_single_1mmDrill, F.Cu at (144.4, 117.9)
- added REF**: SolderWirePad_single_1mmDrill, Wire_Pads:SolderWirePad_single_1mmDrill, F.Cu at (141.9, 117.9)
- added REF**: SolderWirePad_single_1mmDrill, Wire_Pads:SolderWirePad_single_1mmDrill, F.Cu at (139.3, 117.9)
- added REF**: SolderWirePad_single_1mmDrill, Wire_Pads:SolderWirePad_single_1mmDrill, F.Cu at (147.0, 120.4)
- added REF**: SolderWirePad_single_1mmDrill, Wire_Pads:SolderWirePad_single_1mmDrill, F.Cu at (136.8, 117.9)
- added REF**: SolderWirePad_single_1mmDrill, Wire_Pads:SolderWirePad_single_1mmDrill, F.Cu at (134.3, 117.9)
- added REF**: SolderWirePad_single_1mmDrill, Wire_Pads:SolderWirePad_single_1mmDrill, F.Cu at (131.7, 117.9)
- added REF**: SolderWirePad_single_1mmDrill, Wire_Pads:SolderWirePad_single_1mmDrill, F.Cu at (129.2, 117.9)
- added REF**: SolderWirePad_single_1mmDrill, Wire_Pads:SolderWirePad_single_1mmDrill, F.Cu at (126.6, 117.9)
- added REF**: SolderWirePad_single_1mmDrill, Wire_Pads:SolderWirePad_single_1mmDrill, F.Cu at (124.1, 117.9)
- added REF**: SolderWirePad_single_1mmDrill, Wire_Pads:SolderWirePad_single_1mmDrill, F.Cu at (152.0, 115.4)
- added REF**: SolderWirePad_single_1mmDrill, Wire_Pads:SolderWirePad_single_1mmDrill, F.Cu at (149.5, 115.4)
- added REF**: SolderWirePad_single_1mmDrill, Wire_Pads:SolderWirePad_single_1mmDrill, F.Cu at (147.0, 115.4)
- added REF**: SolderWirePad_single_1mmDrill, Wire_Pads:SolderWirePad_single_1mmDrill, F.Cu at (144.4, 115.4)
- added REF**: SolderWirePad_single_1mmDrill, Wire_Pads:SolderWirePad_single_1mmDrill, F.Cu at (144.4, 120.4)
- added REF**: SolderWirePad_single_1mmDrill, Wire_Pads:SolderWirePad_single_1mmDrill, F.Cu at (141.9, 115.4)
- added REF**: SolderWirePad_single_1mmDrill, Wire_Pads:SolderWirePad_single_1mmDrill, F.Cu at (139.3, 115.4)
- added REF**: SolderWirePad_single_1mmDrill, Wire_Pads:SolderWirePad_single_1mmDrill, F.Cu at (136.8, 115.4)
- added REF**: SolderWirePad_single_1mmDrill, Wire_Pads:SolderWirePad_single_1mmDrill, F.Cu at (134.3, 115.4)
- added REF**: SolderWirePad_single_1mmDrill, Wire_Pads:SolderWirePad_single_1mmDrill, F.Cu at (131.7, 115.4)
- added REF**: SolderWirePad_single_1mmDrill, Wire_Pads:SolderWirePad_single_1mmDrill, F.Cu at (129.2, 115.4)
- added REF**: SolderWirePad_single_1mmDrill, Wire_Pads:SolderWirePad_single_1mmDrill, F.Cu at (126.6, 115.4)
- added REF**: SolderWirePad_single_1mmDrill, Wire_Pads:SolderWirePad_single_1mmDrill, F.Cu at (124.1, 115.4)
- added REF**: SolderWirePad_single_1mmDrill, Wire_Pads:SolderWirePad_single_1mmDrill, F.Cu at (152.0, 112.8)
- added REF**: SolderWirePad_single_1mmDrill, Wire_Pads:SolderWirePad_single_1mmDrill, F.Cu at (149.5, 112.8)
- added REF**: SolderWirePad_single_1mmDrill, Wire_Pads:SolderWirePad_single_1mmDrill, F.Cu at (141.9, 120.4)
- added REF**: SolderWirePad_single_1mmDrill, Wire_Pads:SolderWirePad_single_1mmDrill, F.Cu at (147.0, 112.8)
- added REF**: SolderWirePad_single_1mmDrill, Wire_Pads:SolderWirePad_single_1mmDrill, F.Cu at (144.4, 112.8)
- added REF**: SolderWirePad_single_1mmDrill, Wire_Pads:SolderWirePad_single_1mmDrill, F.Cu at (141.9, 112.8)
- added REF**: SolderWirePad_single_1mmDrill, Wire_Pads:SolderWirePad_single_1mmDrill, F.Cu at (139.3, 112.8)
- added REF**: SolderWirePad_single_1mmDrill, Wire_Pads:SolderWirePad_single_1mmDrill, F.Cu at (136.8, 112.8)
- added REF**: SolderWirePad_single_1mmDrill, Wire_Pads:SolderWirePad_single_1mmDrill, F.Cu at (134.3, 112.8)
- added REF**: SolderWirePad_single_1mmDrill, Wire_Pads:SolderWirePad_single_1mmDrill, F.Cu at (131.7, 112.8)
- added REF**: SolderWirePad_single_1mmDrill, Wire_Pads:SolderWirePad_single_1mmDrill, F.Cu at (129.2, 112.8)
- added REF**: SolderWirePad_single_1mmDrill, Wire_Pads:SolderWirePad_single_1mmDrill, F.Cu at (126.6, 112.8)
- added REF**: SolderWirePad_single_1mmDrill, Wire_Pads:SolderWirePad_single_1mmDrill, F.Cu at (124.1, 112.8)
- added REF**: SolderWirePad_single_1mmDrill, Wire_Pads:SolderWirePad_single_1mmDrill, F.Cu at (139.3, 120.4)
- added REF**: SolderWirePad_single_1mmDrill, Wire_Pads:SolderWirePad_single_1mmDrill, F.Cu at (152.0, 110.3)
- added REF**: SolderWirePad_single_1mmDrill, Wire_Pads:SolderWirePad_single_1mmDrill, F.Cu at (149.5, 110.3)
- added REF**: SolderWirePad_single_1mmDrill, Wire_Pads:SolderWirePad_single_1mmDrill, F.Cu at (147.0, 110.3)
- added REF**: SolderWirePad_single_1mmDrill, Wire_Pads:SolderWirePad_single_1mmDrill, F.Cu at (144.4, 110.3)
- added REF**: SolderWirePad_single_1mmDrill, Wire_Pads:SolderWirePad_single_1mmDrill, F.Cu at (141.9, 110.3)
- added REF**: SolderWirePad_single_1mmDrill, Wire_Pads:SolderWirePad_single_1mmDrill, F.Cu at (139.3, 110.3)
- added REF**: SolderWirePad_single_1mmDrill, Wire_Pads:SolderWirePad_single_1mmDrill, F.Cu at (136.8, 110.3)
- added REF**: SolderWirePad_single_1mmDrill, Wire_Pads:SolderWirePad_single_1mmDrill, F.Cu at (134.3, 110.3)
- added REF**: SolderWirePad_single_1mmDrill, Wire_Pads:SolderWirePad_single_1mmDrill, F.Cu at (131.7, 110.3)
- added REF**: SolderWirePad_single_1mmDrill, Wire_Pads:SolderWirePad_single_1mmDrill, F.Cu at (129.2, 110.3)
- added REF**: SolderWirePad_single_1mmDrill, Wire_Pads:SolderWirePad_single_1mmDrill, F.Cu at (136.8, 120.4)
- added REF**: SolderWirePad_single_1mmDrill, Wire_Pads:SolderWirePad_single_1mmDrill, F.Cu at (126.6, 110.3)
- added REF**: SolderWirePad_single_1mmDrill, Wire_Pads:SolderWirePad_single_1mmDrill, F.Cu at (124.1, 110.3)
- added REF**: SolderWirePad_single_1mmDrill, Wire_Pads:SolderWirePad_single_1mmDrill, F.Cu at (152.0, 107.7)
- added REF**: SolderWirePad_single_1mmDrill, Wire_Pads:SolderWirePad_single_1mmDrill, F.Cu at (149.5, 107.7)
- added REF**: SolderWirePad_single_1mmDrill, Wire_Pads:SolderWirePad_single_1mmDrill, F.Cu at (147.0, 107.7)
- added REF**: SolderWirePad_single_1mmDrill, Wire_Pads:SolderWirePad_single_1mmDrill, F.Cu at (144.4, 107.7)
- added REF**: SolderWirePad_single_1mmDrill, Wire_Pads:SolderWirePad_single_1mmDrill, F.Cu at (141.9, 107.7)
- added REF**: SolderWirePad_single_1mmDrill, Wire_Pads:SolderWirePad_single_1mmDrill, F.Cu at (139.3, 107.7)
- added REF**: SolderWirePad_single_1mmDrill, Wire_Pads:SolderWirePad_single_1mmDrill, F.Cu at (136.8, 107.7)
- added REF**: SolderWirePad_single_1mmDrill, Wire_Pads:SolderWirePad_single_1mmDrill, F.Cu at (134.3, 107.7)
- added REF**: SolderWirePad_single_1mmDrill, Wire_Pads:SolderWirePad_single_1mmDrill, F.Cu at (134.3, 120.4)
- added REF**: SolderWirePad_single_1mmDrill, Wire_Pads:SolderWirePad_single_1mmDrill, F.Cu at (131.7, 107.7)
- added REF**: SolderWirePad_single_1mmDrill, Wire_Pads:SolderWirePad_single_1mmDrill, F.Cu at (129.2, 107.7)
- added REF**: SolderWirePad_single_1mmDrill, Wire_Pads:SolderWirePad_single_1mmDrill, F.Cu at (126.6, 107.7)
- added REF**: SolderWirePad_single_1mmDrill, Wire_Pads:SolderWirePad_single_1mmDrill, F.Cu at (124.1, 107.7)
- added REF**: SolderWirePad_single_1mmDrill, Wire_Pads:SolderWirePad_single_1mmDrill, F.Cu at (124.1, 105.2)
- added REF**: SolderWirePad_single_1mmDrill, Wire_Pads:SolderWirePad_single_1mmDrill, F.Cu at (160.0, 130.5)
- added REF**: SolderWirePad_single_1mmDrill, Wire_Pads:SolderWirePad_single_1mmDrill, F.Cu at (160.0, 127.9)
- added REF**: SolderWirePad_single_1mmDrill, Wire_Pads:SolderWirePad_single_1mmDrill, F.Cu at (160.0, 125.4)
- added REF**: SolderWirePad_single_1mmDrill, Wire_Pads:SolderWirePad_single_1mmDrill, F.Cu at (160.0, 122.8)
- added REF**: SolderWirePad_single_1mmDrill, Wire_Pads:SolderWirePad_single_1mmDrill, F.Cu at (160.0, 120.3)
- added REF**: SolderWirePad_single_1mmDrill, Wire_Pads:SolderWirePad_single_1mmDrill, F.Cu at (131.7, 120.4)
- added REF**: SolderWirePad_single_1mmDrill, Wire_Pads:SolderWirePad_single_1mmDrill, F.Cu at (160.0, 117.8)
- added REF**: SolderWirePad_single_1mmDrill, Wire_Pads:SolderWirePad_single_1mmDrill, F.Cu at (160.0, 115.2)
- added REF**: SolderWirePad_single_1mmDrill, Wire_Pads:SolderWirePad_single_1mmDrill, F.Cu at (160.0, 112.7)
- added REF**: SolderWirePad_single_1mmDrill, Wire_Pads:SolderWirePad_single_1mmDrill, F.Cu at (160.0, 108.7)
- added REF**: SolderWirePad_single_1mmDrill, Wire_Pads:SolderWirePad_single_1mmDrill, F.Cu at (160.0, 106.2)
- added REF**: SolderWirePad_single_1mmDrill, Wire_Pads:SolderWirePad_single_1mmDrill, F.Cu at (160.0, 103.6)
- added REF**: SolderWirePad_single_1mmDrill, Wire_Pads:SolderWirePad_single_1mmDrill, F.Cu at (160.0, 101.1)
- added REF**: SolderWirePad_single_1mmDrill, Wire_Pads:SolderWirePad_single_1mmDrill, F.Cu at (160.0, 98.5)
- added REF**: SolderWirePad_single_1mmDrill, Wire_Pads:SolderWirePad_single_1mmDrill, F.Cu at (160.0, 96.0)
- added REF**: SolderWirePad_single_1mmDrill, Wire_Pads:SolderWirePad_single_1mmDrill, F.Cu at (160.0, 93.5)
- added SW1: SW_Push, lib_fp:TL3305_Switch, F.Cu at (126.6, 125.0)
- added SW2: SW_Push, lib_fp:TL3305_Switch, F.Cu at (148.4, 125.0)
- moved R2 31.2 mm to (120.0, 76.0), turned to 0 degrees
- moved R4 29.1 mm to (155.0, 78.0), turned to 0 degrees
- moved R3 22.5 mm to (120.0, 74.0), turned to 0 degrees
- moved R5 13.5 mm to (155.0, 76.0), turned to 0 degrees
Connections:
- D1 pad 1: Net-(D1-Pad1) -> +5V
- D2 pad 1: Net-(D2-Pad1) -> +5V
- D3 pad 2: Net-(D3-Pad2) -> +5V
- D4 pad 2: Net-(D4-Pad2) -> +5V
- D5 pad 2: Net-(D5-Pad2) -> +5V
- D6 pad 2: Net-(D6-Pad2) -> +5V
- R2 pad 1: Net-(R2-Pad1) -> Net-(D1-Pad3)
- R2 pad 2: Net-(D3-Pad2) -> Net-(R2-Pad2)
- R3 pad 1: Net-(R2-Pad1) -> Net-(D1-Pad4)
- R3 pad 2: Net-(D4-Pad2) -> Net-(R3-Pad2)
- R4 pad 1: Net-(R2-Pad1) -> Net-(D2-Pad2)
- R4 pad 2: Net-(D5-Pad2) -> Net-(R4-Pad2)
- R5 pad 1: Net-(R2-Pad1) -> Net-(D2-Pad3)
- R5 pad 2: Net-(D6-Pad2) -> Net-(R5-Pad2)
- XA1 pad D10: Net-(D3-Pad1) -> Net-(R7-Pad2)
- XA1 pad D11: Net-(D4-Pad1) -> Net-(R8-Pad2)
- XA1 pad D12: Net-(D5-Pad1) -> Net-(R9-Pad2)
- XA1 pad D13: Net-(D6-Pad1) -> Net-(R10-Pad2)
- XA1 pad D4: Net-(D1-Pad2) -> Net-(R1-Pad2)
- XA1 pad D5: Net-(D1-Pad3) -> Net-(R2-Pad2)
- XA1 pad D6: Net-(D1-Pad4) -> Net-(R3-Pad2)
- XA1 pad D7: Net-(D2-Pad2) -> Net-(R4-Pad2)
- XA1 pad D8: Net-(D2-Pad3) -> Net-(R5-Pad2)
- XA1 pad D9: Net-(D2-Pad4) -> Net-(R6-Pad2)
Routing:
- net +5V: track 0.00 -> 134.1 mm
- net Net-(R1-Pad2): track 0.00 -> 84.1 mm
- net Net-(R2-Pad2): track 0.00 -> 81.3 mm
- net Net-(R3-Pad2): track 0.00 -> 78.9 mm
- net Net-(SW1-Pad1): track 0.00 -> 43.7 mm
- net Net-(R9-Pad2): track 0.00 -> 41.8 mm, vias 0 -> 1
- net Net-(R4-Pad2): track 0.00 -> 40.2 mm
- net Net-(R5-Pad2): track 0.00 -> 38.2 mm
- net Net-(R8-Pad2): track 0.00 -> 37.8 mm, vias 0 -> 1
- net Net-(R6-Pad2): track 0.00 -> 37.1 mm
- net Net-(R7-Pad2): track 0.00 -> 27.1 mm, vias 0 -> 3
- net Net-(D1-Pad3): track 0.00 -> 25.4 mm, vias 0 -> 2
- net Net-(D1-Pad4): track 0.00 -> 25.4 mm, vias 0 -> 2
- net Net-(D2-Pad2): track 0.00 -> 22.0 mm, vias 0 -> 2
- net Net-(D1-Pad2): track 0.00 -> 21.8 mm, vias 0 -> 2
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- added copper zone on B.Cu, net GNDREF
Other:
- board text added: "+5V Rail"
- board text added: "7 6 5 4 3 2 TX 1 RX 0"
- board text added: "@hamster - hamster university https://github.com/cavehamster/classroom"
- board text added: "A0 A1 A2 A3 A4 A5"
- board text added: "Firmware 102 Shield"
- board text added: "GND Rail"
- board text added: "NC IOREF RST 3V3 5V GND GND Vin"
- board text added: "SCL SDA AREF GND 13 12 11 10 9 8"

Commit message: Update readme and images
Parts:
- moved D3 24.1 mm to (125.3, 96.5), turned to 120 degrees
- moved D4 24.0 mm to (149.4, 96.3), turned to 60 degrees
- moved R8 16.3 mm to (145.5, 94.3), turned to 153 degrees
- moved R7 16.1 mm to (129.4, 94.5), turned to 26 degrees
Routing:
- net Net-(R7-Pad2): track 27.1 -> 39.5 mm, vias 3 -> 1
- net Net-(R8-Pad2): track 37.8 -> 27.4 mm
- net Net-(R10-Pad2): track 21.1 -> 23.3 mm
- net Net-(D2-Pad2): track 22.0 -> 23.9 mm
Other:
- board text added: "Ver 1.0 - 2/2018"
- board text removed: "Firmware 102 Shield"
