File: Firmware102/Hardware/DC801 Shield/DC801 Shield.sch (KiCad schematic (older format))
At the start: 19 parts, among them SW1 SW_Push, SW2 SW_Push

Commit message: Adding the presentation and class code Adding gerbers for the shield Adding a simplified schematic for the shield-uno interface Updated KiCad stuff to 5.0 KiCad
Parts:
- D1, D2: symbol device:LED_ARGB -> Device:LED_ARGB
- D3, D4, D5, D6: symbol device:LED -> Device:LED
- R? (x10): symbol device:R -> Device:R
- SW1, SW2: symbol switches:SW_Push -> Switch:SW_Push
Changed lines of the file:
@@
 $EndComp
 $Comp
-L device:LED_ARGB D1
+L Device:LED_ARGB D1
 U 1 1 5A8E3AC3
 P 7820 3000
@@
 $EndComp
 $Comp
-L device:LED_ARGB D2
+L Device:LED_ARGB D2
 U 1 1 5A8E3B35
 P 7820 3890
@@
 	5700 3600 6750 3600
 $Comp
-L device:LED D6
+L Device:LED D6
 U 1 1 5A8ECB4F
 P 7820 5170
@@
 $EndComp
 $Comp
-L device:LED D5
+L Device:LED D5
 U 1 1 5A8ED122
 P 7820 4910
@@
 $EndComp
 $Comp
-L device:LED D4
+L Device:LED D4
 U 1 1 5A8ED12F
 P 7820 4650
@@
 $EndComp
 $Comp
-L device:LED D3
+L Device:LED D3
 U 1 1 5A8ED6F4
 P 7820 4390
@@
 $EndComp
 $Comp
-L switches:SW_Push SW1
+L Switch:SW_Push SW1
 U 1 1 5A8F652F
 P 6400 1990
@@
 $EndComp
 $Comp
-L switches:SW_Push SW2
+L Switch:SW_Push SW2
 U 1 1 5A8F66A8
 P 6390 2360
@@
 	5700 3900 6360 3900
 $Comp
-L device:R R?
+L Device:R R?
 U 1 1 5A8FB17B
 P 7370 4090
@@
 $EndComp
 $Comp
-L device:R R?
+L Device:R R?
 U 1 1 5A8FD190
 P 7370 3890
@@
 $EndComp
 $Comp
-L device:R R?
+L Device:R R?
 U 1 1 5A8FD1EB
 P 7370 3690
@@
 $EndComp
 $Comp
-L device:R R?
+L Device:R R?
 U 1 1 5A8FD31A
 P 7370 3200
@@
 $EndComp
 $Comp
-L device:R R?
+L Device:R R?
 U 1 1 5A8FD320
 P 7370 3000
@@
 $EndComp
 $Comp
-L device:R R?
+L Device:R R?
 U 1 1 5A8FD326
 P 7370 2800
@@
 $EndComp
 $Comp
-L device:R R?
+L Device:R R?
 U 1 1 5A8FDA0B
 P 7370 4390
@@
 $EndComp
 $Comp
-L device:R R?
+L Device:R R?
 U 1 1 5A8FDA85
 P 7370 4650
@@
 $EndComp
 $Comp
-L device:R R?
+L Device:R R?
 U 1 1 5A8FDB11
 P 7370 4910
@@
 $EndComp
 $Comp
-L device:R R?
+L Device:R R?
 U 1 1 5A8FDC69
 P 7370 5170
